File: Solarladeregler.brd (EAGLE design)
At the start: 105.4 x 67 mm, 75 parts, among them CON1 FLATFLEX, IC1 MWL_LT3652LT3652, IC2 LTC3428, IC3 LTC6102, IC4 LTC6102, IC5 TSIC206, Q1 MOSFET, Q2 BSS138, X1 PN87520-S

Commit message: all files
Parts:
- moved SL3 1.27 mm to (17.1, 45.7)
Changed lines of the file:
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@@
 <element name="C14" library="rcl" package="C0805" value="100nF" x="87.63" y="10.16" rot="R270"/>
 <element name="R10" library="rcl" package="R0805" value="4,7k" x="77.47" y="8.89" rot="R270"/>
-<element name="SL3" library="con-amp-quick" package="02P" value="" x="18.415" y="45.72" rot="R270">
-<attribute name="OC_NEWARK" value="unknown" x="18.415" y="45.72" size="1.778" layer="27" rot="R270" display="off"/>
-<attribute name="MPN" value="" x="18.415" y="45.72" size="1.778" layer="27" rot="R270" display="off"/>
-<attribute name="MF" value="" x="18.415" y="45.72" size="1.778" layer="27" rot="R270" display="off"/>
-<attribute name="OC_FARNELL" value="unknown" x="18.415" y="45.72" size="1.778" layer="27" rot="R270" display="off"/>
+<element name="SL3" library="con-amp-quick" package="02P" value="" x="17.145" y="45.72" rot="R270">
+<attribute name="OC_NEWARK" value="unknown" x="17.145" y="45.72" size="1.778" layer="27" rot="R270" display="off"/>
+<attribute name="MPN" value="" x="17.145" y="45.72" size="1.778" layer="27" rot="R270" display="off"/>
+<attribute name="MF" value="" x="17.145" y="45.72" size="1.778" layer="27" rot="R270" display="off"/>
+<attribute name="OC_FARNELL" value="unknown" x="17.145" y="45.72" size="1.778" layer="27" rot="R270" display="off"/>
 </element>
 <element name="R11" library="rcl" package="R0805" value="22k" x="26.035" y="47.625" rot="R90"/>
@@
 <contactref element="SL3" pad="1"/>
 <contactref element="R11" pad="1"/>
-<wire x1="18.415" y1="46.99" x2="26.035" y2="46.675" width="0" layer="19" extent="1-1"/>
+<wire x1="17.145" y1="46.99" x2="26.035" y2="46.675" width="0" layer="19" extent="1-1"/>
 <wire x1="37.38" y1="23.8" x2="26.035" y2="46.675" width="0" layer="19" extent="1-1"/>
 </signal>
@@
 <contactref element="D7" pad="1"/>
 <contactref element="R27" pad="2"/>
-<wire x1="18.415" y1="44.45" x2="56.2" y2="23.03" width="0" layer="19" extent="1-1"/>
-<wire x1="13.97" y1="34.29" x2="18.415" y2="44.45" width="0" layer="19" extent="1-1"/>
+<wire x1="17.145" y1="44.45" x2="56.2" y2="23.03" width="0" layer="19" extent="1-1"/>
+<wire x1="13.97" y1="34.29" x2="17.145" y2="44.45" width="0" layer="19" extent="1-1"/>
 <wire x1="5.08" y1="27.94" x2="13.97" y2="34.29" width="0" layer="19" extent="1-1"/>
 <wire x1="5.08" y1="22.86" x2="5.08" y2="27.94" width="0" layer="19" extent="1-1"/>

Commit message: TSIC 206
resistor +capacitor
Parts:
- added C18: 10nF, rcl:C0805
- added C19: 100nF, rcl:C0805
- added R28: 10k, rcl:R0805
- moved IC5 2.54 mm to (49.5, 36.8)
Connections:
- new net N$53: C18.2, IC5.2, R28.2
- net GND: now also C18.1, C19.2
- net N$50: now also R28.1; no longer IC5.2
- net N$52: now also C19.1
Changed lines of the file:
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@@
 </element>
 <element name="R27" library="rcl" package="PT-10" value="10k" x="16.51" y="29.21" rot="R180"/>
-<element name="IC5" library="linear" package="SO08" value="TSIC206" x="46.99" y="36.83"/>
+<element name="IC5" library="linear" package="SO08" value="TSIC206" x="49.53" y="36.83"/>
+<element name="R28" library="rcl" package="R0805" value="10k" x="54.61" y="36.83" rot="R90"/>
+<element name="C18" library="rcl" package="C0805" value="10nF" x="57.15" y="36.83" rot="R90"/>
+<element name="C19" library="rcl" package="C0805" value="100nF" x="59.69" y="36.83" rot="R270"/>
 </elements>
 <signals>
@@
 <contactref element="CON1" pad="DB2"/>
 <contactref element="R27" pad="1"/>
+<contactref element="C18" pad="1"/>
 <contactref element="IC5" pad="1"/>
+<contactref element="C19" pad="2"/>
 <wire x1="41.91" y1="46.99" x2="42.41" y2="48.34" width="0" layer="19" extent="1-1"/>
 </signal>
@@
 <contactref element="D7" pad="1"/>
 <contactref element="R27" pad="2"/>
-<wire x1="17.145" y1="44.45" x2="56.2" y2="23.03" width="0" layer="19" extent="1-1"/>
-<wire x1="13.97" y1="34.29" x2="17.145" y2="44.45" width="0" layer="19" extent="1-1"/>
+<wire x1="13.97" y1="34.29" x2="56.2" y2="23.03" width="0" layer="19" extent="1-1"/>
+<wire x1="17.145" y1="44.45" x2="13.97" y2="34.29" width="0" layer="19" extent="1-1"/>
 <wire x1="5.08" y1="27.94" x2="13.97" y2="34.29" width="0" layer="19" extent="1-1"/>
 <wire x1="5.08" y1="22.86" x2="5.08" y2="27.94" width="0" layer="19" extent="1-1"/>
@@
 </signal>
 <signal name="N$50">
-<contactref element="IC5" pad="2"/>
 <contactref element="µC" pad="35"/>
-<wire x1="46.38" y1="31.2" x2="46.355" y2="34.23" width="0" layer="19" extent="1-1"/>
+<contactref element="R28" pad="1"/>
+<wire x1="46.38" y1="31.2" x2="54.61" y2="35.88" width="0" layer="19" extent="1-1"/>
 </signal>
 <signal name="N$52">
 <contactref element="IC5" pad="4"/>
 <contactref element="µC" pad="32"/>
-<wire x1="48.98" y1="28.6" x2="48.895" y2="34.23" width="0" layer="19" extent="1-1"/>
+<contactref element="C19" pad="1"/>
+<wire x1="51.435" y1="34.23" x2="59.69" y2="37.78" width="0" layer="19" extent="1-1"/>
+<wire x1="48.98" y1="28.6" x2="51.435" y2="34.23" width="0" layer="19" extent="1-1"/>
+</signal>
+<signal name="N$53">
+<contactref element="R28" pad="2"/>
+<contactref element="IC5" pad="2"/>
+<contactref element="C18" pad="2"/>
+<wire x1="54.61" y1="37.78" x2="57.15" y2="37.78" width="0" layer="19" extent="1-1"/>
+<wire x1="48.895" y1="34.23" x2="54.61" y2="37.78" width="0" layer="19" extent="1-1"/>
 </signal>
 </signals>
